File: ADV728xM_EVAL_SMA-MINISAS_MX8Mx.sch (KiCad schematic (older format))
At the start: 13 parts, among them J1 142-0701-801, J2 142-0701-801, J3 142-0701-801, J4 142-0701-801, J5 Conn_01x04_Male, J6 Conn_01x04_Male, J7 Conn_01x02_Male, J8 Conn_01x02_Male, U1 1-84953-5, U2 NLSX5014DTR2G

Commit message: Add unsaved schematic
Parts:
- removed U1: 1-84953-5, footprints:TE_1-84953-5, symbol 1-84953-5:1-84953-5
- added H1, H2, H3, H4: MountingHole, MountingHole:MountingHole_3.2mm_M3, symbol Mechanical:MountingHole
- added J9: 1888863-4, footprints:TE_1888863-4, symbol 1888863-4:1888863-4
- renumbered U2 to U1
Connections:
- net labels added: +5V, I2C_SCL_1V8, I2C_SDA_1V8, MCLK_1V8, PWDN_1V8, nRST_1V8
- net labels removed: GPIO0_1V8, GPIO1_1V8, I2C_SCL, I2C_SDA
- wire segments 64 -> 91
- no-connect marks 2 -> 6
Other:
- moved on the sheet: R1
